Commit message: container added, states finished

File: robots/iiwa.urdf.xacro (robot description, xacro)
@@ -25,7 +25,5 @@
   <xacro:include filename="$(find iiwa)/urdf/robot/iiwa/lbr_iiwa.xacro"/>
    <!-- tool -->
-<!--
-  <xacro:include filename="$(find logimat_description)/urdf/tool/roll_scan.urdf.xacro"/>
--->
+  <xacro:include filename="$(find iiwa)/urdf/tool/gripper/gripper_camera_connector/gripper_camera_connector.urdf.xacro"/>
   <!-- Construct the miiwa from parts -->
   <!-- Base frame to anchor the robot in the world -->
@@ -35,4 +33,7 @@
 		<origin xyz="0 0 0" rpy="0.0 0.0 0.0"/>
   </xacro:lbr_iiwa>
+  <xacro:gripper_camera_connector name="gripper" parent_link="lbr_iiwa_link_7">
+    <origin xyz="0 0 ${iiwa_flange_height}" rpy="0.0 0.0 0.0"/>
+  </xacro:gripper_camera_connector>
   <!-- tool -->
 <!--
@@ -40,4 +41,4 @@
 		<origin xyz="0 0 ${iiwa_flange_height}" rpy="0.0 0.0 0.0"/>
   </xacro:roll_scan_v0>
--->
+ -->
 </robot>

File: urdf/tool/gripper/gripper_camera_connector/gripper.urdf.xacro (robot description, xacro)
@@ -1,6 +1,6 @@
 <?xml version="1.0"?>
 <robot xmlns:xacro="http://ros.org/wiki/xacro">
-   <xacro:include filename="$(find hercules_description)/urdf/gripper/gripper.transmission.xacro" />
-    <xacro:include filename="$(find hercules_description)/urdf/gripper/gripper.gazebo.xacro" />
+   <xacro:include filename="$(find iiwa)/urdf/tool/gripper/gripper_camera_connector/gripper.transmission.xacro" />
+    <xacro:include filename="$(find iiwa)/urdf/tool/gripper/gripper_camera_connector/gripper.gazebo.xacro" />
 	<xacro:macro name="gripper_v0"  params="name parent *origin">
     <joint name="${name}_1_joint" type="prismatic">

File: urdf/tool/gripper/mako_3d/mako_3d.urdf.xacro (robot description, xacro)
@@ -5,10 +5,10 @@
 xmlns:xacro="http://ros.org/wiki/xacro">
   <!-- Import all Gazebo-customization elements, including Gazebo colors -->
-  <xacro:include filename="$(find iiwa7_description)/urdf/mako_3d/mako_3d.gazebo.xacro" />
+  <xacro:include filename="$(find iiwa)/urdf/tool/gripper/mako_3d/mako_3d.gazebo.xacro" />
   <xacro:property name="pi" value="3.1415926535897931" />
   <xacro:macro name="mako_3d_visual" params="name color">
      <visual>
        <geometry>
-          <mesh filename="package://iiwa7_description/meshes/mako_3d/visual/mako_3d_link/${name}.stl" />
+          <mesh filename="package://iiwa/meshes/mako_3d/visual/mako_3d_link/${name}.stl" />
        </geometry>
        <material name="${color}"/>
@@ -18,5 +18,5 @@
      <collision>
        <geometry>
-          <mesh filename="package://iiwa7_description/meshes/mako_3d/collision/mako_3d_link/${name}.stl" />
+          <mesh filename="package://iiwa/meshes/mako_3d/collision/mako_3d_link/${name}.stl" />
        </geometry>
        <material name="${color}"/>

File: urdf/tool/gripper/mako_3d/mako_3d_standalone.urdf.xacro (robot description, xacro)
@@ -7,6 +7,6 @@
 <!-- The following included files set up definitions of parts of the robot body -->
 <!-- schunk wsg50 -->
-<xacro:include filename="$(find iiwa7_description)/urdf/mako_3d/mako_3d.urdf.xacro" />
-<xacro:include filename="$(find iiwa7_description)/urdf/materials.xacro" />
+<xacro:include filename="$(find iiwa)/urdf/tool/gripper/mako_3d/mako_3d.urdf.xacro" />
+<xacro:include filename="$(find iiwa)/urdf/tool/gripper/materials.xacro" />
 <link name="base_link"/>
 <xacro:mako_3d name="mako_3d" parent_link="base_link" hardware_interface="none">
