Commit message: solved orientaion

File: robots/logimat_env.urdf.xacro (robot description, xacro)
@@ -7,5 +7,5 @@
   <xacro:arg name="wing_down" default="true"/>
   <xacro:arg name="wing_up" default="false"/>
-  <xacro:arg name="miiwa" default="true"/>
+  <xacro:arg name="iiwa" default="true"/>
   <xacro:arg name="overhead" default="false"/>
   <xacro:arg name="safety" default="false"/>
@@ -18,5 +18,5 @@
   <link name="world"/>
 	<xacro:scene name="euroc_env" parent="world">
-		<origin xyz="0.0 0.0 0.0" rpy="0 0 0"/>
+		<origin xyz="-0.85 0.0 0.0" rpy="0 0 0"/>
 	</xacro:scene>
 </robot>
